Commit message: created moving averaged position controller

File: objects/sphere_with_restitution.urdf (robot description, URDF)
Before this commit: robot urdf_robot, 1 links, 0 joints
Links:
- link baseLink: geometry collision mesh filename=textured_sphere_smooth.obj scale=0.08 0.08 0.01; visual mesh filename=textured_sphere_smooth.obj scale=0.08 0.08 0.01

Commit message: might need to switch to velocity control

File: objects/sphere_with_restitution.urdf (robot description, URDF)
Before this commit: robot urdf_robot, 1 links, 0 joints
Links:
- link baseLink: mass .1 -> 1.2
