Commit message: rectified visual+collision geometry transform in panda_chef urdf

File: franka_panda_chef/panda_chef.urdf (robot description, URDF)
Before this commit: robot panda, 14 links, 13 joints
Joints:
- joint panda_hand_joint: origin xyz=0 0 0 rpy=0 0 -0.785398163397 -> xyz=0 0 0 rpy=0 0 0

Commit message: need to get working example

File: franka_panda_chef/panda_chef.urdf (robot description, URDF)
Before this commit: robot panda, 14 links, 13 joints
Links:
- link pan: mass 0.5 -> 0.1
Joints:
- joint panda_joint2: limit lower=-1.8326 upper=1.8326 effort=87 velocity=2.1750 -> lower=-.8326 upper=.8326 effort=87 velocity=2.1750

File: objects/sphere_with_restitution.urdf (robot description, URDF)
Before this commit: robot urdf_robot, 1 links, 0 joints
Links:
- link baseLink: mass 1.2 -> 0.2; geometry collision cylinder length=0.02 radius=0.08; visual mesh filename=textured_sphere_smooth.obj scale=0.08 0.08 0.02
