Commit message: deleted some older environments just to focus on robot chef env. USE THIS GIT HASH TO RECOVER OLDER FILES

File: panda_chef/urdf/panda_chef.urdf (robot description, URDF)
Before this commit: robot panda, 14 links, 13 joints
Joints:
- joint panda_joint2: limit lower=-.8326 upper=.8326 effort=87 velocity=2.1750 -> lower=-.3326 upper=.4326 effort=87 velocity=2.1750
- joint panda_joint4: limit lower=-3.1416 upper=0.0 effort=87 velocity=2.1750 -> lower=-2.5 upper=-1.0 effort=87 velocity=2.1750

File: panda_chef/urdf/sphere_with_restitution.urdf (robot description, URDF)
Before this commit: robot urdf_robot, 1 links, 0 joints
Links:
- link baseLink: mass 0.2 -> 0.1; geometry collision mesh filename=textured_sphere_smooth.obj scale=0.08 0.08 0.02; visual cylinder length=0.02 radius=0.08
