Commit message: updated the panda model with a new pan, has annoying issues still

File: panda_chef/urdf/pan.urdf (robot description, URDF)
Before this commit: robot panda, 1 links, 0 joints
Links:
- link pan: geometry collision cylinder length=0.02 radius=0.12; collision cylinder length=0.185 radius=0.011
