Commit message: added the axes, updated initial pancake position to offset the pancake from the pan

File: panda_chef/urdf/sphere_with_restitution.urdf (robot description, URDF)
Before this commit: robot urdf_robot, 1 links, 0 joints
Links:
- link baseLink: geometry collision cylinder length=0.02 radius=0.08; visual cylinder length=0.02 radius=0.08
